Commit message: Update amr.urdf.xacro

File: urdf/amr.urdf.xacro (robot description, xacro)
@@ -1,16 +1,28 @@
 <?xml version="1.0"?>
 <robot name="amr" xmlns:xacro="http://www.ros.org/wiki/xacro">
-        <link name="world">
-            <origin xyz="0 0 0" rpy="0 0 0"/>
-        </link>
+        <!--<link name="world"/>
         <joint name="dummy" type="fixed">
             <parent link="world"/>
             <child link="amr_body"/>
-        </joint>
+        </joint>-->
+        <!-- wheel params -->
+        <xacro:property name="radius" value="0.1"/>
+        <xacro:property name="height_w" value="0.06"/>
+        <xacro:property name="mass_w" value="30"/>
+        <!-- rialzo params -->
+        <xacro:property name="height_r" value="0.072"/>
+        <xacro:property name="width_r" value="0.925"/>
+        <xacro:property name="depth_r" value="0.8862"/>
+        <xacro:property name="mass_r" value="160"/>
+        <!--body params-->
+        <xacro:property name="height_b" value="0.2579"/>
+        <xacro:property name="width_b" value="1.3008"/>
+        <xacro:property name="depth_b" value="0.9008"/>
+        <xacro:property name="mass_b" value="70"/>
         <link name="left_wheel">
             <inertial>
                 <origin xyz="0 -0.37 -0.1" rpy="0 0 0"/>
-                <mass value="2"/>
-                <inertia ixx="0.1" ixy="0.1" ixz="0.1" iyy="0.1" iyz="0.1" izz="0.1"/>
+                <mass value="${mass_w}"/>
+                <inertia ixx="${mass_w*(3*radius*radius+height_w*height_w)/12}" ixy="0" ixz="0" iyy="${mass_w*(3*radius*radius+height_w*height_w)/12}" iyz="0" izz="${mass_w*radius*radius/2}"/>
             </inertial>
             <visual>
@@ -38,6 +50,6 @@
             <inertial>
                 <origin xyz="0 0.37 -0.1" rpy="0 0 0"/>
-                <mass value="2"/>
-                <inertia ixx="0.1" ixy="0.1" ixz="0.1" iyy="0.1" iyz="0.1" izz="0.1"/>
+                <mass value="${mass_w}"/>
+                <inertia ixx="${mass_w*(3*radius*radius+height_w*height_w)/12}" ixy="0" ixz="0" iyy="${mass_w*(3*radius*radius+height_w*height_w)/12}" iyz="0" izz="${mass_w*radius*radius/2}"/>
             </inertial>
             <visual>
@@ -65,6 +77,6 @@
             <inertial>
                 <origin xyz="0 0 0" rpy="0 0 0"/>
-                <mass value="250"/>
-                <inertia ixx="0.1" ixy="0.1" ixz="0.1" iyy="0.1" iyz="0.1" izz="0.1"/>
+                <mass value="${mass_b}"/>
+                <inertia ixx="${mass_b*(height_b*height_b+depth_b*depth_b)/12}" ixy="0" ixz="0" iyy="${mass_b*(height_b*height_b+width_b*width_b)/12}" iyz="0" izz="${mass_b*(width_b*width_b+depth_b*depth_b)/12}"/>
             </inertial>
             <visual>
@@ -84,6 +96,6 @@
             <inertial>
                 <origin xyz="0 0 0" rpy="0 0 0"/>
-                <mass value="10"/>
-                <inertia ixx="0.1" ixy="0.1" ixz="0.1" iyy="0.1" iyz="0.1" izz="0.1"/>
+                <mass value="${mass_r}"/>
+                <inertia ixx="${mass_r*(height_r*height_r+depth_r*depth_r)/12}" ixy="0" ixz="0" iyy="${mass_r*(height_r*height_r+width_r*width_r)/12}" iyz="0" izz="${mass_r*(width_r*width_r+depth_r*depth_r)/12}"/>
             </inertial>
             <visual>
@@ -104,5 +116,5 @@
             <child link="left_wheel"/>
             <origin xyz="0 0.37 0.1" rpy="0 0 0"/>
-            <limit velocity="0.35" effort="100"/>
+            <limit effort="10000" velocity="0.35"/>
             <axis xyz="0 1 0"/>
         </joint>
@@ -111,5 +123,5 @@
             <child link="right_wheel"/>
             <origin xyz="0 -0.37 0.1" rpy="0 0 0"/>
-            <limit velocity="0.35" effort="100"/>
+            <limit effort="10000" velocity="0.35"/>
             <axis xyz="0 1 0"/>
         </joint>
@@ -157,5 +169,5 @@
                   <controlPeriod>0.001</controlPeriod>
                   <robotSimType>gazebo_ros_control/DefaultRobotHWSim</robotSimType>
-                  <legacyModeNS>true</legacyModeNS>
+                  <legacyModeNS>false</legacyModeNS>
             </plugin>
             <plugin name='diff_drive' filename='libgazebo_ros_diff_drive.so'>
@@ -166,5 +178,5 @@
                 <wheelDiameter>0.2</wheelDiameter>
                 <!-- Limits -->
-                <wheelTorque>1000</wheelTorque>
+                <wheelTorque>10000</wheelTorque>
                 <wheelAcceleration>0.6</wheelAcceleration>
                 <!-- Output -->

Commit message: Update amr.urdf.xacro

File: urdf/amr.urdf.xacro (robot description, xacro)
@@ -1,23 +1,18 @@
 <?xml version="1.0"?>
 <robot name="amr" xmlns:xacro="http://www.ros.org/wiki/xacro">
-        <!--<link name="world"/>
-        <joint name="dummy" type="fixed">
-            <parent link="world"/>
-            <child link="amr_body"/>
-        </joint>-->
         <!-- wheel params -->
         <xacro:property name="radius" value="0.1"/>
         <xacro:property name="height_w" value="0.06"/>
-        <xacro:property name="mass_w" value="30"/>
+        <xacro:property name="mass_w" value="1"/>
         <!-- rialzo params -->
         <xacro:property name="height_r" value="0.072"/>
         <xacro:property name="width_r" value="0.925"/>
         <xacro:property name="depth_r" value="0.8862"/>
-        <xacro:property name="mass_r" value="160"/>
+        <xacro:property name="mass_r" value="1"/>
         <!--body params-->
         <xacro:property name="height_b" value="0.2579"/>
         <xacro:property name="width_b" value="1.3008"/>
         <xacro:property name="depth_b" value="0.9008"/>
-        <xacro:property name="mass_b" value="70"/>
+        <xacro:property name="mass_b" value="1"/>
         <link name="left_wheel">
             <inertial>
@@ -39,6 +34,6 @@
                     <friction>
                         <ode>
-                            <mu>0.8</mu>
-                            <mu2>0.8</mu2>
+                            <mu>0.5</mu>
+                            <mu2>0.5</mu2>
                         </ode>
                     </friction>
@@ -66,6 +61,6 @@
                     <friction>
                         <ode>
-                            <mu>0.8</mu>
-                            <mu2>0.8</mu2>
+                            <mu>0.5</mu>
+                            <mu2>0.5</mu2>
                         </ode>
                     </friction>
@@ -88,5 +83,5 @@
             <collision>
                 <geometry>
-                    <mesh filename="package://amr/collision/amr_body.stl" scale="0.001 0.001 0.001"/>
+                    <mesh filename="package://amr/collision/amr_body_simp.stl" scale="0.001 0.001 0.001"/>
                 </geometry>
                 <origin xyz="0 0 0" rpy="0 0 0"/>
@@ -107,15 +102,64 @@
             <collision>
                 <geometry>
-                    <mesh filename="package://amr/collision/amr_rialzo.stl" scale="0.001 0.001 0.001"/>
-                </geometry>
-                <origin xyz="0 0 0" rpy="0 0 0"/>
-            </collision>
-        </link>
+                    <mesh filename="package://amr/collision/amr_rialzo_simp.stl" scale="0.001 0.001 0.001"/>
+                </geometry>
+                <origin xyz="0 0 0" rpy="0 0 0"/>
+            </collision>
+        </link>
+        <link name="laser_front">
+            <inertial>
+            <origin xyz="-0.37 -0.57 -0.17" rpy="0 0 0"/>
+                <mass value="0.005"/>
+                <inertia ixx="0.0005" ixy="0" ixz="0" iyy="0.0005" iyz="0" izz="0.0005"/>
+            </inertial>
+            <visual>
+                <geometry>
+                    <mesh filename="package://amr/visual/laser_front.dae" scale="0.001 0.001 0.001"/>
+                </geometry>
+                <origin xyz="-0.37 -0.57 -0.17" rpy="0 0 0"/>
+            </visual>
+            <collision>
+                <geometry>
+                    <mesh filename="package://amr/collision/laser_front.stl" scale="0.001 0.001 0.001"/>
+                </geometry>
+                <origin xyz="-0.37 -0.57 -0.17" rpy="0 0 0"/>
+            </collision>
+        </link>
+        <link name="laser_back">
+            <inertial>
+            <origin xyz="0.37 0.57 -0.17" rpy="0 0 0"/>
+                <mass value="0.005"/>
+                <inertia ixx="0.0005" ixy="0" ixz="0" iyy="0.0005" iyz="0" izz="0.0005"/>
+            </inertial>
+            <visual>
+                <geometry>
+                    <mesh filename="package://amr/visual/laser_back.dae" scale="0.001 0.001 0.001"/>
+                </geometry>
+                <origin xyz="0.37 0.57 -0.17" rpy="0 0 0"/>
+            </visual>
+            <collision>
+                <geometry>
+                    <mesh filename="package://amr/collision/laser_back.stl" scale="0.001 0.001 0.001"/>
+                </geometry>
+                <origin xyz="0.37 0.57 -0.17" rpy="0 0 0"/>
+            </collision>
+        </link>
+        <joint name="laser_front_joint" type="fixed">
+            <parent link="amr_body"/>
+            <child link="laser_front"/>
+            <origin xyz="0.37 0.57 0.17" rpy="0 0 0"/>
+        </joint>
+        <joint name="laser_back_joint" type="fixed">
+            <parent link="amr_body"/>
+            <child link="laser_back"/>
+            <origin xyz="-0.37 -0.57 0.17" rpy="0 0 0"/>
+        </joint>
         <joint name="left_wheel_joint" type="continuous">
             <parent link="amr_body"/>
             <child link="left_wheel"/>
             <origin xyz="0 0.37 0.1" rpy="0 0 0"/>
-            <limit effort="10000" velocity="0.35"/>
+            <limit effort="100" velocity="1.5"/>
             <axis xyz="0 1 0"/>
+            <dynamics damping="0.5" friction="0.1" />
         </joint>
         <joint name="right_wheel_joint" type="continuous">
@@ -123,6 +167,7 @@
             <child link="right_wheel"/>
             <origin xyz="0 -0.37 0.1" rpy="0 0 0"/>
-            <limit effort="10000" velocity="0.35"/>
+            <limit effort="100" velocity="1.5"/>
             <axis xyz="0 1 0"/>
+            <dynamics damping="0.5" friction="0.1" />
         </joint>
         <joint name="rialzo_joint" type="prismatic">
@@ -130,6 +175,13 @@
             <child link="amr_rialzo"/>
             <origin xyz="0 0 0" rpy="0 0 0"/>
-            <limit lower="0" upper="0.06" velocity="0.02" effort="1000"/>
+            <limit lower="0" upper="0.06" velocity="0.02" effort="10"/>
             <axis xyz="0 0 1"/>
+            <dynamics damping="0.1" friction="0.1" />
+        </joint>
+        <link name="base_footprint" />
+        <joint name="footprint_joint" type="fixed">
+            <parent link="amr_body"/>
+            <child link="base_footprint"/>
+            <origin xyz="0 0 0" rpy="0 0 0"/>
         </joint>
         <transmission name="trans_rialzo_joint" >
@@ -165,6 +217,6 @@
         <gazebo>
             <plugin name="gazebo_ros_control" filename="libgazebo_ros_control.so">
-                <robotNamespace>/amr</robotNamespace>
-                  <robotParam>robot_description</robotParam>
+                <robotNamespace>amr</robotNamespace>
+                  <!-- <robotParam>robot_description</robotParam> -->
                   <controlPeriod>0.001</controlPeriod>
                   <robotSimType>gazebo_ros_control/DefaultRobotHWSim</robotSimType>
@@ -178,5 +230,5 @@
                 <wheelDiameter>0.2</wheelDiameter>
                 <!-- Limits -->
-                <wheelTorque>10000</wheelTorque>
+                <wheelTorque>10</wheelTorque>
                 <wheelAcceleration>0.6</wheelAcceleration>
                 <!-- Output -->
@@ -186,5 +238,5 @@
                 <publishWheelTF>true</publishWheelTF>
                 <alwaysOn>true</alwaysOn>
-                <updateRate>100</updateRate>
+                <updateRate>10</updateRate>
                 <legacyMode>false</legacyMode>
                 <commandTopic>cmd_vel</commandTopic>
@@ -192,7 +244,63 @@
                 <publishWheelJointState>true</publishWheelJointState>
                 <rosDebugLevel>na</rosDebugLevel>
-                <odometrySource>world</odometrySource>
+                <odometrySource>encoder</odometrySource>
                 <publishTf>1</publishTf>
             </plugin>
         </gazebo>
+        <gazebo reference="laser_front">
+            <sensor name="laser_front" type="ray">
+                <pose> 0 0 0 0 0 0 </pose>
+                <visualize>true</visualize>
+                <update_rate>1</update_rate>
+                <ray>
+                   <scan>
+                        <horizontal>
+                            <samples>270</samples>
+                            <min_angle>-3.1415</min_angle>
+                            <max_angle>3.1415</max_angle>
+                        </horizontal>
+                    </scan>
+                    <range>
+                        <min>0.289</min>
+                        <max>4</max>
+                        <resolution>0.01</resolution>
+                    </range>
+                </ray>
+                <plugin name="laser_front_controller" filename="libgazebo_ros_laser.so">
+                    <ros>
+                        <argument>~/out:=scan</argument>
+                    </ros>
+                    <output_type>sensor_msgs/LaserScan</output_type>
+                    <frame_name>laser_front</frame_name>
+                </plugin>
+            </sensor>
+        </gazebo>
+        <gazebo reference="laser_back">
+            <sensor name="laser_back" type="ray">
+                <pose> 0 0 0 0 0 0 </pose>
+                <visualize>true</visualize>
+                <update_rate>1</update_rate>
+                <ray>
+                   <scan>
+                        <horizontal>
+                            <samples>270</samples>
+                            <min_angle>0</min_angle>
+                            <max_angle>6.2831</max_angle>
+                        </horizontal>
+                    </scan>
+                    <range>
+                        <min>0.289</min>
+                        <max>4</max>
+                        <resolution>0.01</resolution>
+                    </range>
+                </ray>
+                <plugin name="laser_back_controller" filename="libgazebo_ros_laser.so">
+                    <ros>
+                        <argument>~/out:=scan</argument>
+                    </ros>
+                    <output_type>sensor_msgs/LaserScan</output_type>
+                    <frame_name>laser_back</frame_name>
+                </plugin>
+            </sensor>
+        </gazebo>
 </robot>
